Commit message: 2021/9/2

File: src/turtlebot3/turtlebot3_description/urdf/turtlebot3_waffle.gazebo.xacro (robot description, xacro)
@@ -4,8 +4,9 @@
   <xacro:arg name="camera_visual" default="false"/>
   <xacro:arg name="imu_visual"    default="false"/>
-  <gazebo reference="base_link">
+  <xacro:arg name="robot"         default=""/>
+  <gazebo reference="$(arg robot)base_link">
     <material>Gazebo/DarkGrey</material>
   </gazebo>
-  <gazebo reference="wheel_left_link">
+  <gazebo reference="$(arg robot)wheel_left_link">
     <mu1>0.1</mu1>
     <mu2>0.1</mu2>
@@ -17,5 +18,5 @@
     <material>Gazebo/FlatBlack</material>
   </gazebo>
-  <gazebo reference="wheel_right_link">
+  <gazebo reference="$(arg robot)wheel_right_link">
     <mu1>0.1</mu1>
     <mu2>0.1</mu2>
@@ -27,5 +28,5 @@
     <material>Gazebo/FlatBlack</material>
   </gazebo>
-  <gazebo reference="caster_back_right_link">
+  <gazebo reference="$(arg robot)caster_back_right_link">
     <mu1>0.1</mu1>
     <mu2>0.1</mu2>
@@ -36,5 +37,5 @@
     <material>Gazebo/FlatBlack</material>
   </gazebo>
-  <gazebo reference="caster_back_left_link">
+  <gazebo reference="$(arg robot)caster_back_left_link">
     <mu1>0.1</mu1>
     <mu2>0.1</mu2>
@@ -45,5 +46,5 @@
     <material>Gazebo/FlatBlack</material>
   </gazebo>
-  <gazebo reference="imu_link">
+  <gazebo reference="$(arg robot)imu_link">
     <sensor type="imu" name="imu">
       <always_on>true</always_on>
@@ -56,8 +57,8 @@
       <commandTopic>cmd_vel</commandTopic>
       <odometryTopic>odom</odometryTopic>
-      <odometryFrame>odom</odometryFrame>
+      <odometryFrame>$(arg robot)odom</odometryFrame>
       <odometrySource>world</odometrySource>
       <publishOdomTF>true</publishOdomTF>
-      <robotBaseFrame>base_footprint</robotBaseFrame>
+      <robotBaseFrame>$(arg robot)base_footprint</robotBaseFrame>
       <publishWheelTF>false</publishWheelTF>
       <publishTf>true</publishTf>
@@ -77,6 +78,6 @@
     <plugin name="imu_plugin" filename="libgazebo_ros_imu.so">
       <alwaysOn>true</alwaysOn>
-      <bodyName>imu_link</bodyName>
-      <frameName>imu_link</frameName>
+      <bodyName>$(arg robot)imu_link</bodyName>
+      <frameName>$(arg robot)imu_link</frameName>
       <topicName>imu</topicName>
       <serviceName>imu_service</serviceName>
@@ -102,5 +103,5 @@
     </plugin>
   </gazebo>
-  <gazebo reference="base_scan">
+  <gazebo reference="$(arg robot)base_scan">
     <material>Gazebo/FlatBlack</material>
     <sensor type="ray" name="lds_lfcd_sensor">
@@ -130,9 +131,9 @@
       <plugin name="gazebo_ros_lds_lfcd_controller" filename="libgazebo_ros_laser.so">
         <topicName>scan</topicName>
-        <frameName>base_scan</frameName>
+        <frameName>$(arg robot)base_scan</frameName>
       </plugin>
     </sensor>
   </gazebo>
-  <gazebo reference="camera_rgb_frame">
+  <gazebo reference="$(arg robot)camera_rgb_frame">
     <sensor type="depth" name="realsense_R200">
       <always_on>true</always_on>
@@ -156,5 +157,5 @@
         <updateRate>30.0</updateRate>
         <cameraName>camera</cameraName>
-        <frameName>camera_rgb_optical_frame</frameName>
+        <frameName>$(arg robot)camera_rgb_optical_frame</frameName>
         <imageTopicName>rgb/image_raw</imageTopicName>
         <depthImageTopicName>depth/image_raw</depthImageTopicName>

File: src/turtlebot3/turtlebot3_description/urdf/turtlebot3_waffle.urdf.xacro (robot description, xacro)
@@ -1,17 +1,21 @@
 <?xml version="1.0" ?>
 <robot name="turtlebot3_waffle" xmlns:xacro="http://ros.org/wiki/xacro">
+  <!--↓ノータッチ-->
+  <xacro:arg name="robot"  default=""/>
   <xacro:include filename="$(find turtlebot3_description)/urdf/common_properties.xacro"/>
-  <xacro:include filename="$(find turtlebot3_description)/urdf/turtlebot3_waffle.gazebo.xacro"/>
+  <xacro:include filename="$(find turtlebot3_description)/urdf/turtlebot3_waffle.gazebo.xacro">
+    <xacro:arg name="robot" default="$(arg robot)"/>
+  </xacro:include>
   <xacro:property name="r200_cam_rgb_px" value="0.005"/>
   <xacro:property name="r200_cam_rgb_py" value="0.018"/>
   <xacro:property name="r200_cam_rgb_pz" value="0.013"/>
   <xacro:property name="r200_cam_depth_offset" value="0.01"/>
-  <link name="base_footprint"/>
+  <link name="$(arg robot)base_footprint"/>
   <joint name="base_joint" type="fixed">
-    <parent link="base_footprint"/>
-    <child link="base_link" />
+    <parent link="$(arg robot)base_footprint"/>
+    <child link="$(arg robot)base_link" />
     <origin xyz="0 0 0.010" rpy="0 0 0"/>
   </joint>
-  <link name="base_link">
+  <link name="$(arg robot)base_link">
     <visual>
       <origin xyz="-0.064 0 0.0" rpy="0 0 0"/>
@@ -36,10 +40,10 @@
   </link>
   <joint name="wheel_left_joint" type="continuous">
-    <parent link="base_link"/>
-    <child link="wheel_left_link"/>
+    <parent link="$(arg robot)base_link"/>
+    <child link="$(arg robot)wheel_left_link"/>
     <origin xyz="0.0 0.144 0.023" rpy="-1.57 0 0"/>
     <axis xyz="0 0 1"/>
   </joint>
-  <link name="wheel_left_link">
+  <link name="$(arg robot)wheel_left_link">
     <visual>
       <origin xyz="0 0 0" rpy="1.57 0 0"/>
@@ -64,10 +68,10 @@
   </link>
   <joint name="wheel_right_joint" type="continuous">
-    <parent link="base_link"/>
-    <child link="wheel_right_link"/>
+    <parent link="$(arg robot)base_link"/>
+    <child link="$(arg robot)wheel_right_link"/>
     <origin xyz="0.0 -0.144 0.023" rpy="-1.57 0 0"/>
     <axis xyz="0 0 1"/>
   </joint>
-  <link name="wheel_right_link">
+  <link name="$(arg robot)wheel_right_link">
     <visual>
       <origin xyz="0 0 0" rpy="1.57 0 0"/>
@@ -92,9 +96,9 @@
   </link>
   <joint name="caster_back_right_joint" type="fixed">
-    <parent link="base_link"/>
-    <child link="caster_back_right_link"/>
+    <parent link="$(arg robot)base_link"/>
+    <child link="$(arg robot)caster_back_right_link"/>
     <origin xyz="-0.177 -0.064 -0.004" rpy="-1.57 0 0"/>
   </joint>
-  <link name="caster_back_right_link">
+  <link name="$(arg robot)caster_back_right_link">
     <collision>
       <origin xyz="0 0.001 0" rpy="0 0 0"/>
@@ -112,9 +116,9 @@
   </link>
   <joint name="caster_back_left_joint" type="fixed">
-    <parent link="base_link"/>
-    <child link="caster_back_left_link"/>
+    <parent link="$(arg robot)base_link"/>
+    <child link="$(arg robot)caster_back_left_link"/>
     <origin xyz="-0.177 0.064 -0.004" rpy="-1.57 0 0"/>
   </joint>
-  <link name="caster_back_left_link">
+  <link name="$(arg robot)caster_back_left_link">
     <collision>
       <origin xyz="0 0.001 0" rpy="0 0 0"/>
@@ -132,15 +136,15 @@
   </link>
   <joint name="imu_joint" type="fixed">
-    <parent link="base_link"/>
-    <child link="imu_link"/>
+    <parent link="$(arg robot)base_link"/>
+    <child link="$(arg robot)imu_link"/>
     <origin xyz="0.0 0 0.068" rpy="0 0 0"/>
   </joint>
-  <link name="imu_link"/>
+  <link name="$(arg robot)imu_link"/>
   <joint name="scan_joint" type="fixed">
-    <parent link="base_link"/>
-    <child link="base_scan"/>
+    <parent link="$(arg robot)base_link"/>
+    <child link="$(arg robot)base_scan"/>
     <origin xyz="-0.064 0 0.122" rpy="0 0 0"/>
   </joint>
-  <link name="base_scan">
+  <link name="$(arg robot)base_scan">
     <visual>
       <origin xyz="0 0 0" rpy="0 0 0"/>
@@ -166,8 +170,8 @@
   <joint name="camera_joint" type="fixed">
     <origin xyz="0.064 -0.065 0.094" rpy="0 0 0"/>
-    <parent link="base_link"/>
-    <child link="camera_link"/>
-  </joint>
-  <link name="camera_link">
+    <parent link="$(arg robot)base_link"/>
+    <child link="$(arg robot)camera_link"/>
+  </joint>
+  <link name="$(arg robot)camera_link">
     <visual>
      <origin xyz="0 0 0" rpy="1.57 0 1.57"/>
@@ -193,25 +197,25 @@
   <joint name="camera_rgb_joint" type="fixed">
     <origin xyz="${r200_cam_rgb_px} ${r200_cam_rgb_py} ${r200_cam_rgb_pz}" rpy="0 0 0"/>
-    <parent link="camera_link"/>
-    <child link="camera_rgb_frame"/>
-  </joint>
-  <link name="camera_rgb_frame"/>
+    <parent link="$(arg robot)camera_link"/>
+    <child link="$(arg robot)camera_rgb_frame"/>
+  </joint>
+  <link name="$(arg robot)camera_rgb_frame"/>
   <joint name="camera_rgb_optical_joint" type="fixed">
     <origin xyz="0 0 0" rpy="-1.57 0 -1.57"/>
-    <parent link="camera_rgb_frame"/>
-    <child link="camera_rgb_optical_frame"/>
-  </joint>
-  <link name="camera_rgb_optical_frame"/>
+    <parent link="$(arg robot)camera_rgb_frame"/>
+    <child link="$(arg robot)camera_rgb_optical_frame"/>
+  </joint>
+  <link name="$(arg robot)camera_rgb_optical_frame"/>
   <joint name="camera_depth_joint" type="fixed">
     <origin xyz="${r200_cam_rgb_px} ${r200_cam_rgb_py + r200_cam_depth_offset} ${r200_cam_rgb_pz}" rpy="0 0 0"/>
-    <parent link="camera_link"/>
-    <child link="camera_depth_frame"/>
-  </joint>
-  <link name="camera_depth_frame"/>
+    <parent link="$(arg robot)camera_link"/>
+    <child link="$(arg robot)camera_depth_frame"/>
+  </joint>
+  <link name="$(arg robot)camera_depth_frame"/>
   <joint name="camera_depth_optical_joint" type="fixed">
     <origin xyz="0 0 0" rpy="-1.57 0 -1.57"/>
-    <parent link="camera_depth_frame"/>
-    <child link="camera_depth_optical_frame"/>
-  </joint>
-  <link name="camera_depth_optical_frame"/>
+    <parent link="$(arg robot)camera_depth_frame"/>
+    <child link="$(arg robot)camera_depth_optical_frame"/>
+  </joint>
+  <link name="$(arg robot)camera_depth_optical_frame"/>
 </robot>

Commit message: git pullは重要やね

File: src/turtlebot3/turtlebot3_description/urdf/turtlebot3_waffle.gazebo.xacro (robot description, xacro)
@@ -4,9 +4,8 @@
   <xacro:arg name="camera_visual" default="false"/>
   <xacro:arg name="imu_visual"    default="false"/>
-  <xacro:arg name="robot"         default=""/>
-  <gazebo reference="$(arg robot)base_link">
+  <gazebo reference="base_link">
     <material>Gazebo/DarkGrey</material>
   </gazebo>
-  <gazebo reference="$(arg robot)wheel_left_link">
+  <gazebo reference="wheel_left_link">
     <mu1>0.1</mu1>
     <mu2>0.1</mu2>
@@ -18,5 +17,5 @@
     <material>Gazebo/FlatBlack</material>
   </gazebo>
-  <gazebo reference="$(arg robot)wheel_right_link">
+  <gazebo reference="wheel_right_link">
     <mu1>0.1</mu1>
     <mu2>0.1</mu2>
@@ -28,5 +27,5 @@
     <material>Gazebo/FlatBlack</material>
   </gazebo>
-  <gazebo reference="$(arg robot)caster_back_right_link">
+  <gazebo reference="caster_back_right_link">
     <mu1>0.1</mu1>
     <mu2>0.1</mu2>
@@ -37,5 +36,5 @@
     <material>Gazebo/FlatBlack</material>
   </gazebo>
-  <gazebo reference="$(arg robot)caster_back_left_link">
+  <gazebo reference="caster_back_left_link">
     <mu1>0.1</mu1>
     <mu2>0.1</mu2>
@@ -46,5 +45,5 @@
     <material>Gazebo/FlatBlack</material>
   </gazebo>
-  <gazebo reference="$(arg robot)imu_link">
+  <gazebo reference="imu_link">
     <sensor type="imu" name="imu">
       <always_on>true</always_on>
@@ -57,8 +56,8 @@
       <commandTopic>cmd_vel</commandTopic>
       <odometryTopic>odom</odometryTopic>
-      <odometryFrame>$(arg robot)odom</odometryFrame>
+      <odometryFrame>odom</odometryFrame>
       <odometrySource>world</odometrySource>
       <publishOdomTF>true</publishOdomTF>
-      <robotBaseFrame>$(arg robot)base_footprint</robotBaseFrame>
+      <robotBaseFrame>base_footprint</robotBaseFrame>
       <publishWheelTF>false</publishWheelTF>
       <publishTf>true</publishTf>
@@ -78,6 +77,6 @@
     <plugin name="imu_plugin" filename="libgazebo_ros_imu.so">
       <alwaysOn>true</alwaysOn>
-      <bodyName>$(arg robot)imu_link</bodyName>
-      <frameName>$(arg robot)imu_link</frameName>
+      <bodyName>imu_link</bodyName>
+      <frameName>imu_link</frameName>
       <topicName>imu</topicName>
       <serviceName>imu_service</serviceName>
@@ -103,5 +102,5 @@
     </plugin>
   </gazebo>
-  <gazebo reference="$(arg robot)base_scan">
+  <gazebo reference="base_scan">
     <material>Gazebo/FlatBlack</material>
     <sensor type="ray" name="lds_lfcd_sensor">
@@ -131,9 +130,9 @@
       <plugin name="gazebo_ros_lds_lfcd_controller" filename="libgazebo_ros_laser.so">
         <topicName>scan</topicName>
-        <frameName>$(arg robot)base_scan</frameName>
+        <frameName>base_scan</frameName>
       </plugin>
     </sensor>
   </gazebo>
-  <gazebo reference="$(arg robot)camera_rgb_frame">
+  <gazebo reference="camera_rgb_frame">
     <sensor type="depth" name="realsense_R200">
       <always_on>true</always_on>
@@ -157,5 +156,5 @@
         <updateRate>30.0</updateRate>
         <cameraName>camera</cameraName>
-        <frameName>$(arg robot)camera_rgb_optical_frame</frameName>
+        <frameName>camera_rgb_optical_frame</frameName>
         <imageTopicName>rgb/image_raw</imageTopicName>
         <depthImageTopicName>depth/image_raw</depthImageTopicName>

File: src/turtlebot3/turtlebot3_description/urdf/turtlebot3_waffle.urdf.xacro (robot description, xacro)
@@ -1,21 +1,17 @@
 <?xml version="1.0" ?>
 <robot name="turtlebot3_waffle" xmlns:xacro="http://ros.org/wiki/xacro">
-  <!--↓ノータッチ-->
-  <xacro:arg name="robot"  default=""/>
   <xacro:include filename="$(find turtlebot3_description)/urdf/common_properties.xacro"/>
-  <xacro:include filename="$(find turtlebot3_description)/urdf/turtlebot3_waffle.gazebo.xacro">
-    <xacro:arg name="robot" default="$(arg robot)"/>
-  </xacro:include>
+  <xacro:include filename="$(find turtlebot3_description)/urdf/turtlebot3_waffle.gazebo.xacro"/>
   <xacro:property name="r200_cam_rgb_px" value="0.005"/>
   <xacro:property name="r200_cam_rgb_py" value="0.018"/>
   <xacro:property name="r200_cam_rgb_pz" value="0.013"/>
   <xacro:property name="r200_cam_depth_offset" value="0.01"/>
-  <link name="$(arg robot)base_footprint"/>
+  <link name="base_footprint"/>
   <joint name="base_joint" type="fixed">
-    <parent link="$(arg robot)base_footprint"/>
-    <child link="$(arg robot)base_link" />
+    <parent link="base_footprint"/>
+    <child link="base_link" />
     <origin xyz="0 0 0.010" rpy="0 0 0"/>
   </joint>
-  <link name="$(arg robot)base_link">
+  <link name="base_link">
     <visual>
       <origin xyz="-0.064 0 0.0" rpy="0 0 0"/>
@@ -40,10 +36,10 @@
   </link>
   <joint name="wheel_left_joint" type="continuous">
-    <parent link="$(arg robot)base_link"/>
-    <child link="$(arg robot)wheel_left_link"/>
+    <parent link="base_link"/>
+    <child link="wheel_left_link"/>
     <origin xyz="0.0 0.144 0.023" rpy="-1.57 0 0"/>
     <axis xyz="0 0 1"/>
   </joint>
-  <link name="$(arg robot)wheel_left_link">
+  <link name="wheel_left_link">
     <visual>
       <origin xyz="0 0 0" rpy="1.57 0 0"/>
@@ -68,10 +64,10 @@
   </link>
   <joint name="wheel_right_joint" type="continuous">
-    <parent link="$(arg robot)base_link"/>
-    <child link="$(arg robot)wheel_right_link"/>
+    <parent link="base_link"/>
+    <child link="wheel_right_link"/>
     <origin xyz="0.0 -0.144 0.023" rpy="-1.57 0 0"/>
     <axis xyz="0 0 1"/>
   </joint>
-  <link name="$(arg robot)wheel_right_link">
+  <link name="wheel_right_link">
     <visual>
       <origin xyz="0 0 0" rpy="1.57 0 0"/>
@@ -96,9 +92,9 @@
   </link>
   <joint name="caster_back_right_joint" type="fixed">
-    <parent link="$(arg robot)base_link"/>
-    <child link="$(arg robot)caster_back_right_link"/>
+    <parent link="base_link"/>
+    <child link="caster_back_right_link"/>
     <origin xyz="-0.177 -0.064 -0.004" rpy="-1.57 0 0"/>
   </joint>
-  <link name="$(arg robot)caster_back_right_link">
+  <link name="caster_back_right_link">
     <collision>
       <origin xyz="0 0.001 0" rpy="0 0 0"/>
@@ -116,9 +112,9 @@
   </link>
   <joint name="caster_back_left_joint" type="fixed">
-    <parent link="$(arg robot)base_link"/>
-    <child link="$(arg robot)caster_back_left_link"/>
+    <parent link="base_link"/>
+    <child link="caster_back_left_link"/>
     <origin xyz="-0.177 0.064 -0.004" rpy="-1.57 0 0"/>
   </joint>
-  <link name="$(arg robot)caster_back_left_link">
+  <link name="caster_back_left_link">
     <collision>
       <origin xyz="0 0.001 0" rpy="0 0 0"/>
@@ -136,15 +132,15 @@
   </link>
   <joint name="imu_joint" type="fixed">
-    <parent link="$(arg robot)base_link"/>
-    <child link="$(arg robot)imu_link"/>
+    <parent link="base_link"/>
+    <child link="imu_link"/>
     <origin xyz="0.0 0 0.068" rpy="0 0 0"/>
   </joint>
-  <link name="$(arg robot)imu_link"/>
+  <link name="imu_link"/>
   <joint name="scan_joint" type="fixed">
-    <parent link="$(arg robot)base_link"/>
-    <child link="$(arg robot)base_scan"/>
+    <parent link="base_link"/>
+    <child link="base_scan"/>
     <origin xyz="-0.064 0 0.122" rpy="0 0 0"/>
   </joint>
-  <link name="$(arg robot)base_scan">
+  <link name="base_scan">
     <visual>
       <origin xyz="0 0 0" rpy="0 0 0"/>
@@ -170,8 +166,8 @@
   <joint name="camera_joint" type="fixed">
     <origin xyz="0.064 -0.065 0.094" rpy="0 0 0"/>
-    <parent link="$(arg robot)base_link"/>
-    <child link="$(arg robot)camera_link"/>
-  </joint>
-  <link name="$(arg robot)camera_link">
+    <parent link="base_link"/>
+    <child link="camera_link"/>
+  </joint>
+  <link name="camera_link">
     <visual>
      <origin xyz="0 0 0" rpy="1.57 0 1.57"/>
@@ -197,25 +193,25 @@
   <joint name="camera_rgb_joint" type="fixed">
     <origin xyz="${r200_cam_rgb_px} ${r200_cam_rgb_py} ${r200_cam_rgb_pz}" rpy="0 0 0"/>
-    <parent link="$(arg robot)camera_link"/>
-    <child link="$(arg robot)camera_rgb_frame"/>
-  </joint>
-  <link name="$(arg robot)camera_rgb_frame"/>
+    <parent link="camera_link"/>
+    <child link="camera_rgb_frame"/>
+  </joint>
+  <link name="camera_rgb_frame"/>
   <joint name="camera_rgb_optical_joint" type="fixed">
     <origin xyz="0 0 0" rpy="-1.57 0 -1.57"/>
-    <parent link="$(arg robot)camera_rgb_frame"/>
-    <child link="$(arg robot)camera_rgb_optical_frame"/>
-  </joint>
-  <link name="$(arg robot)camera_rgb_optical_frame"/>
+    <parent link="camera_rgb_frame"/>
+    <child link="camera_rgb_optical_frame"/>
+  </joint>
+  <link name="camera_rgb_optical_frame"/>
   <joint name="camera_depth_joint" type="fixed">
     <origin xyz="${r200_cam_rgb_px} ${r200_cam_rgb_py + r200_cam_depth_offset} ${r200_cam_rgb_pz}" rpy="0 0 0"/>
-    <parent link="$(arg robot)camera_link"/>
-    <child link="$(arg robot)camera_depth_frame"/>
-  </joint>
-  <link name="$(arg robot)camera_depth_frame"/>
+    <parent link="camera_link"/>
+    <child link="camera_depth_frame"/>
+  </joint>
+  <link name="camera_depth_frame"/>
   <joint name="camera_depth_optical_joint" type="fixed">
     <origin xyz="0 0 0" rpy="-1.57 0 -1.57"/>
-    <parent link="$(arg robot)camera_depth_frame"/>
-    <child link="$(arg robot)camera_depth_optical_frame"/>
-  </joint>
-  <link name="$(arg robot)camera_depth_optical_frame"/>
+    <parent link="camera_depth_frame"/>
+    <child link="camera_depth_optical_frame"/>
+  </joint>
+  <link name="camera_depth_optical_frame"/>
 </robot>
